File: RTL8723DS-BreakOut.kicad_sch (KiCad schematic)
At the start: 25 parts, among them J1 PWR_TER, J2 PWR_CONN, J3 WL_ACT_CONN, J4 BT_ACT_CONN, J5 CLK_CONN, J6 INT_SIG_CONN, J7 BT_CONN, J8 WL_CONN

Commit message: Update design
Parts:
- removed J5: CLK_CONN, Connector_PinHeader_2.54mm:PinHeader_1x03_P2.54mm_Vertical, symbol Connector_Generic:Conn_01x03
- added J5: SUSCLK_CONN, Connector_PinHeader_2.54mm:PinHeader_1x02_P2.54mm_Vertical, symbol Connector_Generic:Conn_01x02
- added J9: XTAL_CONN, Connector_PinHeader_2.54mm:PinHeader_1x02_P2.54mm_Vertical, symbol Connector_Generic:Conn_01x02
- AE1: footprint RF_Antenna:Texas_SWRA117D_2.4GHz_Right -> RF_Antenna:Texas_SWRA117D_2.4GHz_Left
Connections:
- net BT_WAKE_HOST: now also J7.10 (Pin_10); no longer J7.11 (Pin_11)
- net GND: now also RF1.1 (GND), RF1.20 (GND), RF1.3 (GND), RF1.31 (GND), RF1.33 (GND), RF1.36 (GND), RF1.45 (GND), J5.2 (Pin_2), J9.2 (Pin_2); no longer AE1.2 (Shield), RF1.1,3,20,31,33,36,45 (GND)
- net HOST_WAKE_BT: now also J7.11 (Pin_11); no longer J7.10 (Pin_10)
- net MAIN_XTAL_IN: now also J9.1 (Pin_1)
- net SD_CLK: now also J8.6 (Pin_6); no longer J8.7 (Pin_7)
- net SD_CMD: now also J8.5 (Pin_5); no longer J8.6 (Pin_6)
- net SD_D0: now also J8.7 (Pin_7); no longer J8.2 (Pin_2)
- net SD_D1: now also J8.8 (Pin_8); no longer J8.3 (Pin_3)
- net SD_D2: now also J8.3 (Pin_3); no longer J8.4 (Pin_4)
- net SD_D3: now also J8.4 (Pin_4); no longer J8.5 (Pin_5)
- net SUSCLK_IN: now also J5.1 (Pin_1)
- net WL_HOST_WAKE: now also J8.2 (Pin_2); no longer J8.8 (Pin_8)
- no-connect marks 1 -> 2
Other:
- moved on the sheet: J6
